File: pcb/esp-daikin/kicad-src/esp-daikin-r1p0.kicad_sch (KiCad schematic)
At the start: 31 parts, among them J1 PH_01x05, J2 PinHeader 1x02, U1 ESP32-C3-MINI-1, U3 AOZ1280CI

Commit message: pcb: Update daikin-esp
 - Add test-point for GPIO9
Parts:
- added TP4: JDB_CTRL, TestPoint:TestPoint_Pad_D1.0mm, symbol Connector:TestPoint_Alt
Connections:
- net at U1.23 (GPIO9): now also TP4.1
Other:
- moved on the sheet: C1, C2, C3, C5, C6, C7, D2, D3, J1, J2, L1, R1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
