File: pcb/esp-daikin/kicad-src/esp-daikin-r1p0.kicad_sch (KiCad schematic)
At the start: 32 parts, among them J1 PH_01x05, J2 PinHeader 1x02, U1 ESP32-C3-MINI-1, U3 AOZ1280CI

Commit message: pcb.esp-daikin: Update PNs
Parts:
- C1: LCSC (none) -> C19702; MFG YAGEO -> (none); Mfg Yageo -> (none); PN CC0603MRX5R8BB106 -> (none); lcsc C596327 -> (none)
- C2, C5: LCSC (none) -> C16772; MFG YAGEO -> (none); Mfg Yageo -> (none); PN CC0402KRX5R8BB224 -> (none); lcsc C326836 -> (none)
- C3: LCSC (none) -> C15850; MFG YAGEO -> (none); Mfg Yageo -> (none); PN CC0603MRX5R8BB106 -> (none); lcsc C596327 -> (none)
- C6: LCSC (none) -> C106862; MFG YAGEO -> (none); Mfg Yageo -> (none); PN CC0402KRX7R9BB333 -> (none); lcsc C106862 -> (none)
- C7: LCSC (none) -> C59461; MFG YAGEO -> (none); Mfg Yageo -> (none); PN CC0603MRX5R8BB226 -> (none); lcsc C596327 -> (none)
- D2: LCSC (none) -> C965791; MFG XINGLIGHT -> (none); PN XL-1005UOC -> (none); lcsc C965791 -> (none)
- D3: LCSC (none) -> C8523
- L1: LCSC (none) -> C63166; MFG APV -> (none); PN ANR4020T4R7M -> (none); lcsc C6364800 -> (none)
- R1, R3: LCSC (none) -> C25905; MFG YAGEO -> (none); PN RC0402FR-075K1L -> (none); lcsc C105872 -> (none)
- R12, R13: LCSC (none) -> C25879; MFG YAGEO -> (none); PN RC0402FR-072K2L -> (none); lcsc C114762 -> (none)
- R14: LCSC (none) -> C25117; MFG YAGEO -> (none); PN RC0402FR-07470RL -> (none); lcsc C114877 -> (none)
- R4: LCSC (none) -> C26956; MFG YAGEO -> (none); PN RC0402FR-0725K5L -> (none); lcsc C138065 -> (none)
- R7: LCSC (none) -> C25897; MFG YAGEO -> (none); PN RC0402FR-07115KL -> (none); lcsc C137961 -> (none)
- U1: LCSC (none) -> C2934569; MFG Espressif Systems -> (none); PN ESP32-C3-MINI-1-H4 -> (none); lcsc C2934569 -> (none)
- U3: LCSC (none) -> C41240
