File: pcb/esp-daikin/kicad-src/esp-daikin-r1p1.kicad_pcb (KiCad board)
At the start: 2 copper layers, 28.6 x 30 mm, 37 parts, among them J1 PH_01x05, J2 PinHeader 1x02, U1 ESP32-C3-MINI-1, U3 AOZ1280CI

Commit message: pcb.daikin-esp: Add r1p1
 - Add GPIO9 test-point to enter UART boot
Parts:
- removed kibuzzard-65E1B005: G***, kibuzzard-65E1B005
- removed kibuzzard-65E9962C: G***, kibuzzard-65E9962C
- added kibuzzard-663027A7: G***, kibuzzard-663027A7, F.Cu at (163.6, 86.3)
- added kibuzzard-663027CC: G***, kibuzzard-663027CC, F.Cu at (164.7, 87.6)
